File: cta-thermistor/cta-thermistor.kicad_sch (KiCad schematic)
At the start: 38 parts, among them Con1 100u, Q1 TIP120, Q2 BC557, U1 OP07, U2 LM358

Commit message: I used the wrong footprint for the OpAmps
I mistakenly selected a wide footprint. Used the opportunity to do some improvements on the PCB layout.
Parts:
- U1, U2: footprint Package_DIP:DIP-8_W10.16mm_LongPads -> Package_DIP:DIP-8_W7.62mm_LongPads
Changed lines of the file:
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@@
 			)
 		)
-		(property "Footprint" "Package_DIP:DIP-8_W10.16mm_LongPads"
+		(property "Footprint" "Package_DIP:DIP-8_W7.62mm_LongPads"
 			(at 205.74 74.93 0)
 			(effects
@@
 			)
 		)
-		(property "Footprint" "Package_DIP:DIP-8_W10.16mm_LongPads"
+		(property "Footprint" "Package_DIP:DIP-8_W7.62mm_LongPads"
 			(at 106.68 115.57 0)
 			(effects
@@
 			)
 		)
-		(property "Footprint" "Package_DIP:DIP-8_W10.16mm_LongPads"
+		(property "Footprint" "Package_DIP:DIP-8_W7.62mm_LongPads"
 			(at 242.57 68.58 0)
 			(effects
@@
 			)
 		)
-		(property "Footprint" "Package_DIP:DIP-8_W10.16mm_LongPads"
+		(property "Footprint" "Package_DIP:DIP-8_W7.62mm_LongPads"
 			(at 195.58 135.89 0)
 			(effects
