File: anem-offset/anem-offset.kicad_sch (KiCad schematic)
At the start: 34 parts, among them IC1 LM336, Q1 TIP120, U1 LM324, U2 LM358

Commit message: Pequenas correções e melhorias
 * Furos de montagem
 * Valores 'mais corretos' dos componentes.
Parts:
- CI1: value C -> 1n
- RV2, Rd2, Rs1, Rs2: value 1k -> 10k
- Rd1: value 1k -> 20k
- Rf1: value 10k -> 15k
- Rref1: value 1.2k -> 3.9k
Changed lines of the file:
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@@
 			)
 		)
-		(property "Value" "1k"
+		(property "Value" "10k"
 			(at 74.93 126.9999 0)
 			(effects
@@
 			)
 		)
-		(property "Value" "1k"
+		(property "Value" "20k"
 			(at 107.95 146.0499 0)
 			(effects
@@
 			)
 		)
-		(property "Value" "1k"
+		(property "Value" "10k"
 			(at 116.84 68.58 90)
 			(effects
@@
 			)
 		)
-		(property "Value" "1k"
+		(property "Value" "10k"
 			(at 107.95 160.0199 0)
 			(effects
@@
 			)
 		)
-		(property "Value" "C"
+		(property "Value" "1n"
 			(at 161.29 45.7199 0)
 			(effects
@@
 			)
 		)
-		(property "Value" "1k"
+		(property "Value" "10k"
 			(at 116.84 58.42 90)
 			(effects
@@
 			)
 		)
-		(property "Value" "1.2k"
+		(property "Value" "3.9k"
 			(at 54.61 109.2199 0)
 			(effects
@@
 			)
 		)
-		(property "Value" "10k"
+		(property "Value" "15k"
 			(at 138.43 151.13 90)
 			(effects
